File: HWProj/synth_module_test/design.sch (EAGLE design)
At the start: 39 parts, among them IC1 LM311N, IC10 TL071P, IC11 TL071P, IC12 TL071P, IC13 TL071P, IC2 TL071P, IC3 TL071P, IC4 TL071P, IC5 LM311N, IC8 TL071P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

Commit message: begin designing entire schematic, added power
Parts:
- TM2: value 10k -> 100k
Other:
- note added: "max 1Vrms input"
Changed lines of the file:
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@@
 <part name="SUPPLY15" library="supply2" library_urn="urn:adsk.eagle:library:372" deviceset="V-" device=""/>
 <part name="GND18" library="HyTechSymbols" deviceset="GND" device=""/>
-<part name="TM2" library="HyTechDevices" deviceset="TRIMPOT" device="" value="10k"/>
+<part name="TM2" library="HyTechDevices" deviceset="TRIMPOT" device="" value="100k"/>
 <part name="U$2" library="HyTechDevices" deviceset="PAM8302A_ADAFRUIT" device=""/>
 <part name="GND10" library="HyTechSymbols" deviceset="GND" device=""/>
@@
 <text x="20.32" y="104.14" size="1.778" layer="150">-100mV to 100mV signal range</text>
 <text x="205.74" y="35.56" size="1.778" layer="150">volume control</text>
+<text x="228.6" y="22.86" size="1.778" layer="150">max 1Vrms input</text>
 </plain>
 <instances>

Commit message: changed value of volume control pot at speaker stage to 50k
Parts:
- TM2: value 100k -> 50k
Changed lines of the file:
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@@
 <part name="SUPPLY15" library="supply2" library_urn="urn:adsk.eagle:library:372" deviceset="V-" device=""/>
 <part name="GND18" library="HyTechSymbols" deviceset="GND" device=""/>
-<part name="TM2" library="HyTechDevices" deviceset="TRIMPOT" device="" value="100k"/>
+<part name="TM2" library="HyTechDevices" deviceset="TRIMPOT" device="" value="50k"/>
 <part name="U$2" library="HyTechDevices" deviceset="PAM8302A_ADAFRUIT" device=""/>
 <part name="GND10" library="HyTechSymbols" deviceset="GND" device=""/>
