File: HWProj/design.brd (EAGLE design)
At the start: 149.8 x 123.1 mm, 89 parts, among them IC1 LM311N, IC10 TL071P, IC11 TL071P, IC12 TL071P, IC13 TL071P, IC14 TL071P, IC15 TL071P, IC16 LM311N, IC17 TL071P, IC18 TL071P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

Commit message: post-prototype evaluation revisions
Parts:
- moved PAUSE 3.12 mm to (70.0, 12.4)
- moved PLAY 3.12 mm to (70.0, 17.5)
- moved REC 3.12 mm to (70.0, 7.37)
- moved POWER 3.12 mm to (70.0, 22.6)
- moved POT2_EXT 2.54 mm to (71.1, 92.7)
- moved POT3_EXT 2.54 mm to (81.3, 92.7)
- moved TM7 2.54 mm to (66.0, 87.6)
- moved U$5 2.54 mm to (118.1, 25.4)
- moved U$7 1.27 mm to (120.7, 16.5)
- moved POT1_EXT 1.27 mm to (61.0, 92.7)
- moved TM6 1.27 mm to (55.9, 87.6)
- moved TM2 1.27 mm to (87.6, 94.0)
- moved TM5 1.27 mm to (76.2, 87.6)
Routing:
- net BANDPASS_OUT: track 82.6 -> 76.1 mm
- net HIGHPASS_OUT: track 67.6 -> 73.2 mm
- net RECORD: track 18.2 -> 21.6 mm
- net GND: track 451.7 -> 448.7 mm
- net PAUSE: track 13.5 -> 16.1 mm
- net PLAY: track 8.15 -> 10.7 mm
- net N$32: track 50.1 -> 47.5 mm
- net N$29: track 38.6 -> 36.3 mm
- net N$22: track 49.2 -> 47.2 mm, vias 1 -> 0
- net N$25: track 69.7 -> 71.5 mm
- net N$1: track 35.6 -> 34.4 mm
- net SHUNT_ADC_POLL: track 138.2 -> 139.0 mm
- net N$20: track 57.7 -> 58.2 mm
Other:
- board text added: "DPAN02E-15"
- board text added: "M2"
- board text added: "M3"
- board text added: "M5"
- board text added: "buttons"
- board text removed: "boost converter"
- board text removed: "button connections ->"
